Commit message: update fix the robot model

File: robotic_programming_hw5/two_link_description/urdf/myrobot.urdf (robot description, URDF)
Before this commit: robot pi_robot, 9 links, 8 joints
Joints:
- joint base_link__link_01: limit lower=-3.14 upper=3.14 effort=1000.0 velocity=0.5 -> lower=-3.14 upper=3.14 effort=100 velocity=0.5
- joint base_link__link_04: limit lower=-3.14 upper=3.14 effort=1000.0 velocity=0.5 -> lower=-3.14 upper=3.14 effort=100 velocity=0.5
- joint base_link__link_07: limit lower=-3.14 upper=3.14 effort=1000.0 velocity=0.5 -> lower=-3.14 upper=3.14 effort=100 velocity=0.5; origin xyz=0 0 2.65 -> xyz=0 0 1.2

Commit message: update

File: robotic_programming_hw5/two_link_description/urdf/myrobot.urdf (robot description, URDF)
Before this commit: robot pi_robot, 9 links, 8 joints
Links:
- link link6: geometry collision box size=0.2 0.2 1.4; visual box size=0.2 0.2 1.4
Joints:
- removed joint base_link__link_01
- removed joint base_link__link_02
- removed joint base_link__link_03
- removed joint base_link__link_04
- removed joint base_link__link_05
- removed joint base_link__link_06
- removed joint base_link__link_07
- removed joint base_link__link_08
- added joint connect1: type fixed, parent link2, child link3, origin xyz=0 0 0.001
- added joint connect2: type fixed, parent link3, child link4, origin xyz=0 0 0.001
- added joint connect3: type fixed, parent link5, child link6, origin xyz=0 0 0.001
- added joint connect4: type fixed, parent link6, child link7, origin xyz=0 0 0.001
- added joint connect5: type fixed, parent link8, child link9, origin xyz=0 0 0.001
- added joint move_arm1: type revolute, parent link4, child link5, origin xyz=0 0 1.9, axis 0 1 0, limit lower=-2 upper=2 effort=100 velocity=0.5
- added joint move_arm2: type revolute, parent link7, child link8, origin xyz=0 0 1.2, axis 0 1 0, limit lower=-2 upper=2 effort=100 velocity=0.5
- added joint rotate_around: type revolute, parent link1, child link2, origin xyz=0 0 0, axis 0 0 1, limit lower=-2 upper=2 effort=100 velocity=0.5
